File: PCB/NE2000.kicad_pcb (KiCad board)
At the start: 2 copper layers, 157.4 x 74.2 mm, 56 parts, among them J1 Bus_ISA_16bit, J2 RJ45, J3 BNC, SW1 I/O addr, SW2 ROM cfg, SW3 IRQ, SW4 Medium, SW5 PNP, U1 RTL8019AS, U2 93C64D, U3 SST39SF010, U4 IL1209S, U5 DP8392CN, Y1 20MHz

Commit message: Work in progress
Parts:
- added TR2: PE-85728NL, Transformer_SMD:Transformer_Pulse_H1100NL, F.Cu at (178.4, 90.2)
- C16, C17: footprint Capacitor_SMD:C_1206_3216Metric_Pad1.42x1.75mm_HandSolder -> Capacitor_SMD:C_1210_3225Metric_Pad1.42x2.65mm_HandSolder
- moved U3 87.8 mm to (160.7, 67.9), turned to 270 degrees
- moved C9 82.7 mm to (158.1, 79.6), turned to 90 degrees
- moved U2 25.0 mm to (129.5, 75.6), turned to 90 degrees
- moved C8 15.2 mm to (124.7, 73.0), turned to 180 degrees
- moved R5 7.85 mm to (122.6, 52.3)
- moved R6 7.85 mm to (125.1, 52.3)
- moved R7 7.85 mm to (127.6, 52.3)
- moved R8 7.85 mm to (130.2, 52.3)
- moved SW1 7.85 mm to (122.6, 63.5)
- moved R14 7.73 mm to (137.2, 52.3)
- moved R16 7.73 mm to (142.2, 52.3)
- moved R19 7.73 mm to (175.3, 52.3)
- moved SW3 7.73 mm to (137.2, 63.5)
- moved SW5 7.73 mm to (175.3, 63.5)
- moved R15 7.73 mm to (139.7, 52.3)
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Connections:
- J1 pad 78: +5V -> (no net)
- U1 pad 48: (no net) -> TX-
- U1 pad 49: (no net) -> TX+
- U1 pad 53: (no net) -> CD-
- U1 pad 54: (no net) -> CD+
- U1 pad 55: (no net) -> RX-
- U1 pad 56: (no net) -> RX+
Routing:
- net ~SMEMW: track 190.0 -> 59.5 mm, vias 2 -> 3
- net GND: track 0.00 -> 104.1 mm, vias 12 -> 69
- net BA16: track 144.5 -> 51.4 mm, vias 0 -> 1
- net BA15: track 136.3 -> 44.4 mm
- net A6: track 14.3 -> 82.6 mm, vias 0 -> 2
- net A7: track 13.5 -> 77.3 mm, vias 0 -> 1
- net A5: track 16.1 -> 79.4 mm, vias 0 -> 2
- net A12: track 18.4 -> 80.8 mm, vias 0 -> 2
- net BA14: track 107.5 -> 48.6 mm, vias 0 -> 1
- net A4: track 18.0 -> 76.5 mm, vias 0 -> 1
- net A3: track 19.9 -> 76.9 mm, vias 0 -> 1
- net A2: track 21.8 -> 78.3 mm, vias 0 -> 1
- net A1: track 23.4 -> 75.8 mm, vias 0 -> 1
- net A0: track 22.8 -> 74.0 mm, vias 0 -> 1
- net A13: track 20.3 -> 69.3 mm, vias 0 -> 1
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Other:
- board size 157.4 x 74.2 mm -> 157.4 x 78.5 mm

Commit message: Work in progress
Parts:
- added C18: 47u, Capacitor_SMD:C_1210_3225Metric_Pad1.42x2.65mm_HandSolder, F.Cu at (161.9, 104.4)
- added H3: MountingHole, ISA_BUS_16Bit:Cutline, F.Cu at (116.2, 106.7)
- added H4: MountingHole, ISA_BUS_16Bit:Cutline, F.Cu at (116.2, 118.7)
- added H5: MountingHole, ISA_BUS_16Bit:Cutline, F.Cu at (116.2, 102.9)
- added H6: MountingHole, ISA_BUS_16Bit:Cutline, F.Cu at (116.2, 114.9)
- added H7: MountingHole, ISA_BUS_16Bit:Cutline, F.Cu at (116.2, 116.8)
- added H8: MountingHole, ISA_BUS_16Bit:Cutline, F.Cu at (116.2, 113.0)
- added H9: MountingHole, ISA_BUS_16Bit:Cutline, F.Cu at (116.2, 111.1)
- added R22: 510, Resistor_SMD:R_0805_2012Metric_Pad1.15x1.40mm_HandSolder, F.Cu at (188.0, 87.6)
- added R23: 510, Resistor_SMD:R_0805_2012Metric_Pad1.15x1.40mm_HandSolder, F.Cu at (186.1, 87.6)
- added R25: 510, Resistor_SMD:R_0805_2012Metric_Pad1.15x1.40mm_HandSolder, F.Cu at (188.0, 97.2)
- added R26: 510, Resistor_SMD:R_0805_2012Metric_Pad1.15x1.40mm_HandSolder, F.Cu at (186.1, 97.2)
- C16, C17: value C -> 47u
- moved C16 4.84 mm to (161.9, 97.4), turned to 90 degrees
- moved C7 3.71 mm to (187.7, 102.6), turned to 270 degrees
- moved R4 1.90 mm to (189.2, 79.6)
- moved U4 1.27 mm to (166.4, 97.8)
- moved D1 0.89 mm to (201.9, 97.4)
- moved J2 0.89 mm to (214.2, 73.7)
- moved R21 0.78 mm to (201.9, 103.1)
- moved J3 0.63 mm to (207.6, 99.1)
Connections:
- C7 pad 2: GND -> GNDA
- J1 pad 80: GND -> (no net)
- TR2 pad 10: (no net) -> Net-(TR2-Pad10)
- TR2 pad 12: (no net) -> Net-(R26-Pad2)
- TR2 pad 13: (no net) -> Net-(R25-Pad2)
- TR2 pad 15: (no net) -> Net-(R23-Pad2)
- TR2 pad 16: (no net) -> Net-(R22-Pad2)
- TR2 pad 9: (no net) -> Net-(TR2-Pad9)
- U4 pad 4: GND -> GNDA
- U5 pad 1: (no net) -> Net-(R22-Pad2)
- U5 pad 10: GND -> GNDA
- U5 pad 16: GND -> GNDA
- U5 pad 2: (no net) -> Net-(R23-Pad2)
- U5 pad 3: (no net) -> Net-(R25-Pad2)
- U5 pad 6: (no net) -> Net-(R26-Pad2)
- U5 pad 7: (no net) -> Net-(TR2-Pad10)
- U5 pad 8: (no net) -> Net-(TR2-Pad9)
- U5 pad 9: GND -> GNDA
Routing:
- net LED1: track 0.00 -> 118.1 mm, vias 0 -> 2
- net LED0: track 0.00 -> 96.3 mm, vias 0 -> 2
- net +5V: track 384.6 -> 434.1 mm
- net GNDA: track 0.00 -> 44.4 mm, vias 0 -> 1
- net -9V: track 12.9 -> 52.3 mm, vias 0 -> 1
- net GND: track 104.1 -> 73.0 mm, vias 69 -> 57
- net Net-(TR2-Pad10): track 0.00 -> 20.2 mm
- net Net-(TR2-Pad9): track 0.00 -> 19.3 mm
- net Net-(R26-Pad2): track 0.00 -> 18.6 mm, vias 0 -> 1
- net Net-(R25-Pad2): track 0.00 -> 12.0 mm
- net Net-(R23-Pad2): track 0.00 -> 11.2 mm
- net Net-(R22-Pad2): track 0.00 -> 11.1 mm
- net Net-(D1-Pad2): track 0.00 -> 11.0 mm
- net Net-(J2-Pad9): track 0.00 -> 5.39 mm
- net Net-(J2-Pad11): track 0.00 -> 5.29 mm
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- added copper zone on F.Cu, net -9V
- added copper zone on B.Cu, net GNDA
Other:
- board size 157.4 x 78.5 mm -> 156.8 x 78.5 mm

Commit message: Work in progress
Parts:
- added R24: 270, Resistor_SMD:R_0805_2012Metric_Pad1.15x1.40mm_HandSolder, F.Cu at (176.5, 99.5)
- added R27: 270, Resistor_SMD:R_0805_2012Metric_Pad1.15x1.40mm_HandSolder, F.Cu at (174.6, 99.5)
- renumbered R15 to R10, R16 to R11, R17 to R12, R18 to R13, R9 to R14, R10 to R15, R11 to R16, R12 to R17, R13 to R18, R14 to R9, SW3 to SW2, SW4 to SW3, SW2 to SW4
Routing:
- net TPOUT+: track 0.00 -> 78.3 mm, vias 0 -> 2
- net TPOUT-: track 0.00 -> 74.1 mm, vias 0 -> 2
- net TPIN-: track 0.00 -> 64.1 mm, vias 0 -> 2
- net TPIN+: track 0.00 -> 64.1 mm, vias 0 -> 2
- net GND: track 73.0 -> 124.1 mm, vias 57 -> 84
- net RX-: track 0.00 -> 37.2 mm, vias 0 -> 2
- net CD-: track 0.00 -> 36.8 mm, vias 0 -> 2
- net RX+: track 0.00 -> 36.6 mm, vias 0 -> 2
- net CD+: track 0.00 -> 36.2 mm, vias 0 -> 2
- net TX+: track 0.00 -> 30.1 mm, vias 0 -> 2
- net TX-: track 0.00 -> 27.2 mm, vias 0 -> 2
- net Net-(J2-Pad3): track 0.00 -> 21.5 mm, vias 0 -> 1
- net Net-(J2-Pad1): track 0.00 -> 13.9 mm
- net Net-(J2-Pad6): track 0.00 -> 12.0 mm
- net Net-(J2-Pad2): track 0.00 -> 11.4 mm
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- added copper zone on B.Cu, net GND
- added copper zone on F.Cu, net GND
Other:
- board text added: "27C256 27C512"
- board text added: "R5..R19 10Kx16"

Commit message: Minor changes
Connections:
- U1 pad 64: (no net) -> GND
Routing:
- net GND: track 124.1 -> 135.2 mm, vias 84 -> 110

Commit message: Work in progress
Parts:
- added C19: 10n 1kV, Capacitor_SMD:C_1206_3216Metric_Pad1.42x1.75mm_HandSolder, F.Cu at (203.0, 109.2)
- added Q1: PMBT2222, Package_TO_SOT_SMD:SOT-23, F.Cu at (160.1, 96.6)
- added R28: 0, Resistor_SMD:R_0805_2012Metric_Pad1.15x1.40mm_HandSolder, F.Cu at (205.0, 54.6)
- added R29: 0, Resistor_SMD:R_0805_2012Metric_Pad1.15x1.40mm_HandSolder, F.Cu at (203.1, 117.1)
- added R30: 1M, Resistor_SMD:R_0805_2012Metric_Pad1.15x1.40mm_HandSolder, F.Cu at (203.1, 111.8)
- added R31: 1K, Resistor_SMD:R_0805_2012Metric_Pad1.15x1.40mm_HandSolder, F.Cu at (155.6, 99.2)
- C3, C4: value 1nF 2kV -> 100n; footprint Capacitor_SMD:C_1206_3216Metric_Pad1.42x1.75mm_HandSolder -> Capacitor_SMD:C_0805_2012Metric_Pad1.15x1.40mm_HandSolder
- C5, C6: value 1nF 2kV -> 39p 2kV
- moved C5 11.5 mm to (204.2, 76.4), turned to 270 degrees
- moved C6 7.82 mm to (204.2, 71.2)
- moved C16 2.82 mm to (161.1, 100.1), turned to 180 degrees
- moved R2 1.14 mm to (203.2, 65.9)
- moved C3 0.54 mm to (194.3, 66.8)
- moved C4 0.54 mm to (194.3, 85.6)
- moved C15 0.38 mm to (155.6, 97.2)
Connections:
- C5 pad 1: GND -> Net-(C5-Pad1)
- C5 pad 2: Net-(C5-Pad2) -> Earth
- C6 pad 2: GND -> Earth
- H1 pad 1: GND -> Earth
- H2 pad 1: GND -> Earth
- J2 pad 1: Net-(J2-Pad1) -> Net-(C6-Pad1)
- J2 pad 2: Net-(J2-Pad2) -> Net-(C5-Pad1)
- J2 pad SH: GND -> Earth
- J3 pad 2: GND -> GNDA
- TR1 pad 10: Net-(C5-Pad2) -> (no net)
- TR1 pad 14: Net-(J2-Pad2) -> Net-(C5-Pad1)
- TR1 pad 15: Net-(C6-Pad1) -> (no net)
- TR1 pad 16: Net-(J2-Pad1) -> Net-(C6-Pad1)
- U1 pad 60: (no net) -> Net-(R31-Pad2)
- U4 pad 1: GND -> Net-(Q1-Pad3)
Routing:
- net Net-(R31-Pad2): track 0.00 -> 24.3 mm, vias 0 -> 2
- net Net-(J2-Pad1): track 13.9 -> 0.00 mm
- net Net-(C5-Pad1): track 0.00 -> 11.6 mm
- net Net-(J2-Pad2): track 11.4 -> 0.00 mm
- net Net-(C5-Pad2): track 7.22 -> 0.00 mm
- net Net-(Q1-Pad3): track 0.00 -> 7.11 mm
- net Net-(C6-Pad1): track 6.85 -> 13.9 mm
- net GNDA: track 44.4 -> 50.6 mm
- net +5V: track 429.9 -> 426.3 mm
- net Net-(Q1-Pad1): track 0.00 -> 3.23 mm
- net Net-(J2-Pad9): track 5.39 -> 7.13 mm
- net Net-(J2-Pad3): track 21.5 -> 23.0 mm
- net +12V: track 35.3 -> 34.1 mm
- net LED0: track 94.6 -> 93.4 mm
- net GND: track 135.2 -> 135.3 mm, vias 110 -> 114
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
Commit message: Work in progress
Parts:
- added H10: MountingHole, ISA_BUS_16Bit:Cutline, F.Cu at (116.2, 99.7)
- J3: footprint Connector_Coaxial:BNC_Amphenol_B6252HB-NPP3G-50_Horizontal -> Coax:BNC_shield
- moved C5 3.17 mm to (204.2, 79.6)
- renumbered R25 to R24, R26 to R25, R24 to R26
Routing:
- net Earth: track 0.00 -> 24.6 mm, vias 2 -> 19
- net GNDA: track 50.6 -> 62.2 mm
- net Net-(J2-Pad3): track 23.0 -> 14.9 mm, vias 1 -> 0
- net GND: track 135.3 -> 140.2 mm, vias 114 -> 122
- net Net-(C5-Pad1): track 11.6 -> 15.4 mm
- net +5V: track 426.3 -> 429.4 mm
- net Net-(C6-Pad1): track 13.9 -> 16.6 mm
- net Net-(J2-Pad6): track 12.0 -> 14.4 mm
- net DB12: track 66.5 -> 66.0 mm
- added copper zone on B.Cu, net Earth
- added copper zone on F.Cu, net Earth
Other:
- outline, holes or cut-outs redrawn
- rule trace_min: 0.2 -> 0.127
- board text added: "All switches off for PNP"
- board text added: "Can be cut off for 8 bit operation"
- board text added: "Copyright 2021 Ch. Lehner"
- board text added: "DIY ISA NE2000"
- board text added: "JLCJLCJLCJLC"
- board text added: "SW1 I/O addr 0 0 0 0 300H 0 0 0 1 320H 0 0 1 0 340H 0 0 1 1 360H 1 0 0 0 380H 1 0 0 1 3A0H 1 0 1 0 3C0H 1 0 1 1 3E0H 0 1 0 0 200H 0 1 0 1 220H 0 1 1 0 240H 0 1 1 1 260H 1 1 0 0 280H 1 1 0 1 2A0H 1 1 1 0 2C0H 1 1 1 1 2E0H"
- board text added: "SW2 IRQ 0 0 0 IRQ2 0 0 1 IRQ3 0 1 0 IRQ4 0 1 1 IRQ5 1 0 0 IRQ10 1 0 1 IRQ11 1 1 0 IRQ12 1 1 1 IRQ15"
- board text added: "SW3 Medium 0 0 10BaseT w/ link test 0 1 10BaseT w/o link test 1 0 10Base5 1 1 10Base2"
- board text added: "SW4 Boot ROM 0 0 X X X Disabled 0 1 0 0 0 C000H, 32K 0 1 0 0 1 C800H, 32K 0 1 0 1 0 D000H, 32K 0 1 0 1 1 D800H, 32K 0 1 1 0 0 C000H, 64K 0 1 1 0 1 D000H, 64K 1 0 0 0 0 C000H, 16K 1 0 0 0 1 C400H, 16K 1 0 0 1 0 C800H, 16K 1 0 0 1 1 CC00H, 16K 1 0 1 0 0 D000H, 16K 1 0 1 0 1 D400H, 16K 1 0 1 1 0 D800H, 16K 1 0 1 1 1 DC00H, 16K 1 1 0 0 0 C000H, Paged 1 1 0 0 1 C400H, Paged 1 1 0 1 0 C800H, Paged 1 1 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"
- board text added: "SW5 PNP 0 0 Jumperless PNP mode 0 1 Jumper mode 1 0 Force PNP (no EEPROM) 1 1 illegal"
- board text added: "https://github.com/chregu82/DIY_ISA_NE2000"

Commit message: Minor changes
Parts:
- moved C9 3.77 mm to (154.6, 78.4), turned to 180 degrees
- moved C8 0.65 mm to (125.3, 72.9), turned to 90 degrees
- moved R21 0.49 mm to (201.9, 102.6)
- moved C12 0.37 mm to (132.7, 114.4)
- moved C13 0.25 mm to (141.0, 114.4)
- moved C7 0.25 mm to (188.0, 102.6)
Routing:
- net +5V: track 429.4 -> 447.9 mm
- net GND: track 140.2 -> 131.6 mm, vias 122 -> 120
- net A2: track 79.4 -> 73.7 mm
- net A3: track 77.3 -> 71.7 mm
- net A6: track 83.8 -> 80.2 mm
- net A4: track 75.0 -> 71.8 mm
- net A10: track 55.6 -> 52.4 mm
- net A5: track 79.6 -> 76.4 mm
- net ~SMEMR: track 78.8 -> 76.1 mm
- net A1: track 76.1 -> 73.7 mm
- net A11: track 62.7 -> 60.6 mm
- net A0: track 73.9 -> 75.9 mm
- net TPIN-: track 64.1 -> 62.4 mm
- net TPOUT-: track 74.1 -> 72.3 mm
- net TPIN+: track 64.1 -> 62.3 mm
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Other:
- outline, holes or cut-outs redrawn
- board text added: "Cut traces before braking off"

Commit message: Work in progress
Parts:
- D1: value 1N4150 -> BAS16
- U4: footprint Converter_DCDC:Converter_DCDC_muRata_CRE1xxxxxx3C_THT -> Samac:IL1209S
- moved C16 0.34 mm to (160.8, 100.1)
- moved C18 0.25 mm to (161.7, 104.4)
- turned U4 to 270 degrees
Routing:
- net GND: track 131.6 -> 134.8 mm
Changed lines of the file:
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@@
     (thickness 1.6)
     (drawings 64)
-    (tracks 2086)
+    (tracks 2088)
     (zones 0)
     (modules 78)
@@
   )
   (setup
-    (last_trace_width 0.25)
+    (last_trace_width 0.5)
     (user_trace_width 0.127)
     (user_trace_width 0.5)
@@
     (add_net ~SMEMW)
   )
+  (module Samac:IL1209S (layer F.Cu)
+    (at 166.37 97.79 270)
+    (descr IL1209S-1)
+    (tags "Power Supply")
+    (fp_text reference U4 (at 10.795 -1.27 180) (layer F.SilkS)
+      (effects (font (size 1 1) (thickness 0.15)))
+    )
+    (fp_text value IL1209S (at 3.325 -1.72 90) (layer F.SilkS)
+      (effects (font (size 1 1) (thickness 0.15)))
+    )
+    (fp_arc (start -2.95 0) (end -3 0) (angle -180) (layer F.SilkS) (width 0.2))
+    (fp_arc (start -2.95 0) (end -2.9 0) (angle -180) (layer F.SilkS) (width 0.2))
+    (fp_arc (start -2.95 0) (end -3 0) (angle -180) (layer F.SilkS) (width 0.2))
+    (fp_line (start -3 0) (end -3 0) (layer F.SilkS) (width 0.2))
+    (fp_line (start -2.9 0) (end -2.9 0) (layer F.SilkS) (width 0.2))
+    (fp_line (start -3 0) (end -3 0) (layer F.SilkS) (width 0.2))
+    (fp_line (start -4 3.03) (end -4 -6.47) (layer F.CrtYd) (width 0.1))
+    (fp_line (start 10.65 3.03) (end -4 3.03) (layer F.CrtYd) (width 0.1))
+    (fp_line (start 10.65 -6.47) (end 10.65 3.03) (layer F.CrtYd) (width 0.1))
+    (fp_line (start -4 -6.47) (end 10.65 -6.47) (layer F.CrtYd) (width 0.1))
+    (fp_line (start -2.03 2.03) (end -2.03 -5.47) (layer F.SilkS) (width 0.1))
+    (fp_line (start 9.65 2.03) (end -2.03 2.03) (layer F.SilkS) (width 0.1))
+    (fp_line (start 9.65 -5.47) (end 9.65 2.03) (layer F.SilkS) (width 0.1))
+    (fp_line (start -2.03 -5.47) (end 9.65 -5.47) (layer F.SilkS) (width 0.1))
+    (fp_line (start -2.03 -5.47) (end -2.03 2.03) (layer F.Fab) (width 0.2))
+    (fp_line (start 9.65 -5.47) (end -2.03 -5.47) (layer F.Fab) (width 0.2))
+    (fp_line (start 9.65 2.03) (end 9.65 -5.47) (layer F.Fab) (width 0.2))
+    (fp_line (start -2.03 2.03) (end 9.65 2.03) (layer F.Fab) (width 0.2))
+    (fp_text user %R (at 3.325 -1.72 90) (layer F.Fab)
+      (effects (font (size 1.27 1.27) (thickness 0.254)))
+    )
+    (pad 4 thru_hole circle (at 7.62 0 270) (size 1.32 1.32) (drill 0.77) (layers *.Cu *.Mask)
+      (net 117 GNDA))
+    (pad 3 thru_hole circle (at 5.08 0 270) (size 1.32 1.32) (drill 0.77) (layers *.Cu *.Mask)
+      (net 110 -9V))
+    (pad 2 thru_hole circle (at 2.54 0 270) (size 1.32 1.32) (drill 0.77) (layers *.Cu *.Mask)
+      (net 105 +12V))
+    (pad 1 thru_hole circle (at 0 0 270) (size 1.32 1.32) (drill 0.77) (layers *.Cu *.Mask)
+      (net 125 "Net-(Q1-Pad3)"))
+    (model C:\Users\chregu\Documents\GitHub\DIY_ISA_NE2000\PCB\SamacSys_Parts.3dshapes\IL1209S.stp
+      (at (xyz 0 0 0))
+      (scale (xyz 1 1 1))
+      (rotate (xyz 0 0 0))
+    )
+  )
   (module ISA_BUS_16Bit:BUS_AT_WO_SILKSCREEN (layer F.Cu)
     (at 195.64 123.74)
@@
   )
   (module Capacitor_SMD:C_1210_3225Metric_Pad1.42x2.65mm_HandSolder (layer F.Cu)
-    (at 161.925 104.3575 90)
+    (at 161.671 104.3575 90)
     (descr "Capacitor SMD 1210 (3225 Metric), square (rectangular) end terminal, IPC_7351 nominal with elongated pad for handsoldering. (Body size source: http://www.tortai-tech.com/upload/download/2011102023233369053.pdf), generated with kicad-footprint-generator")
     (tags "capacitor handsolder")
@@
   )
   (module Capacitor_SMD:C_1210_3225Metric_Pad1.42x2.65mm_HandSolder (layer F.Cu)
-    (at 161.1265 100.076 180)
+    (at 160.782 100.076 180)
     (descr "Capacitor SMD 1210 (3225 Metric), square (rectangular) end terminal, IPC_7351 nominal with elongated pad for handsoldering. (Body size source: http://www.tortai-tech.com/upload/download/2011102023233369053.pdf), generated with kicad-footprint-generator")
     (tags "capacitor handsolder")
@@
       (effects (font (size 1 1) (thickness 0.15)))
     )
-    (fp_text value 1N4150 (at -0.001 -2.032 90) (layer F.SilkS)
+    (fp_text value BAS16 (at -0.001 -2.032 90) (layer F.SilkS)
       (effects (font (size 1 1) (thickness 0.15)))
     )
@@
     )
   )
-  (module Converter_DCDC:Converter_DCDC_muRata_CRE1xxxxxx3C_THT (layer F.Cu)
-    (at 166.37 97.79)
-    (descr "Isolated 1W single output DC/DC, http://power.murata.com/data/power/ncl/kdc_cre1.pdf")
-    (tags "Isolated 1W single output DC/DC")
-    (fp_text reference U4 (at 1 10.795) (layer F.SilkS)
-      (effects (font (size 1 1) (thickness 0.15)))
-    )
-    (fp_text value IL1209S (at 2.667 3.81 270) (layer F.SilkS)
-      (effects (font (size 1 1) (thickness 0.15)))
-    )
-    (fp_line (start -1.45 -2.27) (end -1.45 -1.07) (layer F.SilkS) (width 0.12))
-    (fp_line (start -0.25 -2.27) (end -1.45 -2.27) (layer F.SilkS) (width 0.12))
-    (fp_line (start 5.22 9.83) (end -1.38 9.83) (layer F.CrtYd) (width 0.05))
-    (fp_line (start -1.38 -2.2) (end -1.38 9.83) (layer F.CrtYd) (width 0.05))
-    (fp_line (start 5.22 -2.2) (end -1.38 -2.2) (layer F.CrtYd) (width 0.05))
-    (fp_line (start 5.22 -2.2) (end 5.22 9.83) (layer F.CrtYd) (width 0.05))
-    (fp_text user %R (at 3 4 90) (layer F.Fab)
-      (effects (font (size 1 1) (thickness 0.15)))
-    )
-    (fp_line (start -1.13 9.58) (end 4.97 9.58) (layer F.Fab) (width 0.1))
-    (fp_line (start -1.13 -0.95) (end -1.13 9.58) (layer F.Fab) (width 0.1))
-    (fp_line (start -0.13 -1.95) (end 4.97 -1.95) (layer F.Fab) (width 0.1))
-    (fp_line (start -0.13 -1.95) (end -1.13 -0.95) (layer F.Fab) (width 0.1))
-    (fp_line (start 4.97 -1.95) (end 4.97 9.58) (layer F.Fab) (width 0.1))
-    (fp_line (start 5.09 9.7) (end -1.25 9.7) (layer F.SilkS) (width 0.12))
-    (fp_line (start -1.25 -2.07) (end -1.25 9.7) (layer F.SilkS) (width 0.12))
-    (fp_line (start 5.09 -2.07) (end -1.25 -2.07) (layer F.SilkS) (width 0.12))
-    (fp_line (start 5.09 -2.07) (end 5.09 9.7) (layer F.SilkS) (width 0.12))
-    (pad 1 thru_hole rect (at 0 0 270) (size 1.4 1.8) (drill 1) (layers *.Cu *.Mask)
-      (net 125 "Net-(Q1-Pad3)"))
-    (pad 2 thru_hole oval (at 0 2.54 270) (size 1.4 1.8) (drill 1) (layers *.Cu *.Mask)
-      (net 105 +12V))
-    (pad 3 thru_hole oval (at 0 5.08 270) (size 1.4 1.8) (drill 1) (layers *.Cu *.Mask)
-      (net 110 -9V))
-    (pad 4 thru_hole oval (at 0 7.62 270) (size 1.4 1.8) (drill 1) (layers *.Cu *.Mask)
-      (net 117 GNDA))
-    (model ${KISYS3DMOD}/Converter_DCDC.3dshapes/Converter_DCDC_muRata_CRE1xxxxxx3C_THT.wrl
-      (at (xyz 0 0 0))
-      (scale (xyz 1 1 1))
-      (rotate (xyz 0 0 0))
-    )
-  )
   (module Resistor_SMD:R_0805_2012Metric_Pad1.15x1.40mm_HandSolder (layer F.Cu)
     (at 189.23 79.62 90)
@@
   (via (at 122.936 75.819) (size 0.8) (drill 0.4) (layers F.Cu B.Cu) (net 1))
   (via (at 167.64 84.709) (size 0.8) (drill 0.4) (layers F.Cu B.Cu) (net 1))
+  (segment (start 161.097 98.2735) (end 159.2945 100.076) (width 0.5) (layer F.Cu) (net 1))
+  (segment (start 161.097 97.647) (end 161.097 98.2735) (width 0.5) (layer F.Cu) (net 1))
   (segment (start 160.02 90.17) (end 161.925 88.265) (width 0.25) (layer F.Cu) (net 2))
   (segment (start 160.02 92.71) (end 160.02 90.17) (width 0.25) (layer F.Cu) (net 2))
@@
   (segment (start 168.27 100.33) (end 168.97999 101.03999) (width 1) (layer F.Cu) (net 105))
   (segment (start 166.37 100.33) (end 168.27 100.33) (width 1) (layer F.Cu) (net 105))
-  (segment (start 162.868 100.33) (end 162.614 100.076) (width 1) (layer F.Cu) (net 105))
-  (segment (start 166.37 100.33) (end 162.868 100.33) (width 1) (layer F.Cu) (net 105))
+  (segment (start 162.5235 100.33) (end 162.2695 100.076) (width 1) (layer F.Cu) (net 105))
+  (segment (start 166.37 100.33) (end 162.5235 100.33) (width 1) (layer F.Cu) (net 105))
   (segment (start 199.25137 96.52) (end 198.12 96.52) (width 0.25) (layer F.Cu) (net 106))
   (segment (start 200.09 96.52) (end 199.25137 96.52) (width 0.25) (layer F.Cu) (net 106))
@@
   (segment (start 198.12 104.14) (end 201.44 104.14) (width 0.25) (layer F.Cu) (net 109))
   (via (at 185.42 101.6) (size 2) (drill 1) (layers F.Cu B.Cu) (net 110))
-  (segment (start 166.37 102.87) (end 161.925 102.87) (width 1) (layer F.Cu) (net 110))
   (segment (start 184.15 102.87) (end 185.42 101.6) (width 1) (layer B.Cu) (net 110))
   (segment (start 166.37 102.87) (end 184.15 102.87) (width 1) (layer B.Cu) (net 110))
@@
   (segment (start 190.5 99.06) (end 188.265 99.06) (width 0.25) (layer F.Cu) (net 110))
   (segment (start 187.96 98.18) (end 186.055 98.18) (width 0.25) (layer F.Cu) (net 110))
+  (segment (start 166.37 102.87) (end 161.671 102.87) (width 1) (layer F.Cu) (net 110))
   (via (at 172.72 94.615) (size 0.8) (drill 0.4) (layers F.Cu B.Cu) (net 111))
   (via (at 168.91 94.615) (size 0.8) (drill 0.4) (layers F.Cu B.Cu) (net 111))
@@
   (segment (start 149.878472 94.154296) (end 152.222788 91.80998) (width 0.25) (layer B.Cu) (net 116))
   (via (at 187.96 106.045) (size 2) (drill 1) (layers F.Cu B.Cu) (net 117))
-  (segment (start 162.36 105.41) (end 161.925 105.845) (width 1) (layer F.Cu) (net 117))
-  (segment (start 166.37 105.41) (end 162.36 105.41) (width 1) (layer F.Cu) (net 117))
   (segment (start 168.27 105.41) (end 169.54 104.14) (width 1) (layer B.Cu) (net 117))
   (segment (start 166.37 105.41) (end 168.27 105.41) (width 1) (layer B.Cu) (net 117))
@@
   (segment (start 205.74 96.52) (end 207.645 96.52) (width 0.5) (layer F.Cu) (net 117))
   (segment (start 203.835 94.615) (end 205.74 96.52) (width 0.5) (layer F.Cu) (net 117))
+  (segment (start 162.106 105.41) (end 161.671 105.845) (width 1) (layer F.Cu) (net 117))
+  (segment (start 166.37 105.41) (end 162.106 105.41) (width 1) (layer F.Cu) (net 117))
   (segment (start 183.515 93.345) (end 182.69 93.345) (width 0.25) (layer F.Cu) (net 118))
   (segment (start 184.094999 102.236001) (end 184.094999 93.924999) (width 0.25) (layer F.Cu) (net 118))
