File: PCB/NE2000.sch (KiCad schematic (older format))
At the start: 56 parts, among them J1 Bus_ISA_16bit, J2 RJ45, J3 BNC, SW1 I/O addr, SW2 ROM cfg, SW3 IRQ, SW4 Medium, SW5 PNP, U1 RTL8019AS, U2 93C64D, U3 SST39SF010, U4 IL1209S, U5 DP8392CN, Y1 20MHz

Commit message: Work in progress
Parts:
- added TR2: PE-85728NL, Transformer_SMD:Transformer_Pulse_H1100NL, symbol 10Base2:PE-85728NL
- C16, C17: footprint Capacitor_SMD:C_1206_3216Metric_Pad1.42x1.75mm_HandSolder -> Capacitor_SMD:C_1210_3225Metric_Pad1.42x2.65mm_HandSolder
Connections:
- net +5V: no longer J1.78 (+5V)
- net TX-: now reaches U1.48 (TX-)
- net TX-: now also TR2.8
- net TX+: now reaches U1.49 (TX+)
- net TX+: now also TR2.7
- net CD-: now reaches U1.53 (CD-)
- net CD-: now also TR2.2
- net CD+: now reaches U1.54 (CD+)
- net CD+: now also TR2.1
- net RX-: now reaches U1.55 (RX-)
- net RX-: now also TR2.5
- net RX+: now reaches U1.56 (RX+)
- net RX+: now also TR2.4
- no-connect marks 43 -> 44
Changed lines of the file:
@@
 EESchema Schematic File Version 4
+LIBS:NE2000-cache
 EELAYER 30 0
 EELAYER END
@@
 	0    -1   -1   0
 $EndComp
-$Comp
-L power:+5V #PWR0116
-U 1 1 606C34AB
-P 1750 6450
-F 0 "#PWR0116" H 1750 6300 50  0001 C CNN
-F 1 "+5V" V 1765 6578 50  0000 L CNN
-F 2 "" H 1750 6450 50  0001 C CNN
-F 3 "" H 1750 6450 50  0001 C CNN
-	1    1750 6450
-	0    -1   -1   0
-$EndComp
-Wire Wire Line
-	1750 6450 2150 6450
 Text GLabel 2150 1850 0    50   Input ~ 0
 RESET
@@
 F 0 "C17" H 1315 4746 50  0000 L CNN
 F 1 "C" H 1315 4655 50  0000 L CNN
-F 2 "Capacitor_SMD:C_1206_3216Metric_Pad1.42x1.75mm_HandSolder" H 1238 4550 50  0001 C CNN
-F 3 "https://www.mouser.ch/datasheet/2/396/mlcc02_e-1307760.pdf" H 1200 4700 50  0001 C CNN
+F 2 "Capacitor_SMD:C_1210_3225Metric_Pad1.42x2.65mm_HandSolder" H 1238 4550 50  0001 C CNN
+F 3 "https://www.mouser.ch/datasheet/2/281/1/GRM32EC81C476KE15_01A-1988154.pdf" H 1200 4700 50  0001 C CNN
 	1    1200 4700
 	1    0    0    -1
@@
 F 0 "C16" H 1315 2746 50  0000 L CNN
 F 1 "C" H 1315 2655 50  0000 L CNN
-F 2 "Capacitor_SMD:C_1206_3216Metric_Pad1.42x1.75mm_HandSolder" H 1238 2550 50  0001 C CNN
-F 3 "https://www.mouser.ch/datasheet/2/396/mlcc02_e-1307760.pdf" H 1200 2700 50  0001 C CNN
+F 2 "Capacitor_SMD:C_1210_3225Metric_Pad1.42x2.65mm_HandSolder" H 1238 2550 50  0001 C CNN
+F 3 "https://www.mouser.ch/datasheet/2/281/1/GRM32EC81C476KE15_01A-1988154.pdf" H 1200 2700 50  0001 C CNN
 	1    1200 2700
 	1    0    0    -1
@@
 	1    0    0    -1
 $EndComp
+NoConn ~ 2150 6450
+$Comp
+L 10Base2:PE-85728NL TR2
+U 1 1 60779AED
+P 10900 6350
+F 0 "TR2" H 10900 7315 50  0000 C CNN
+F 1 "PE-85728NL" H 10900 7224 50  0000 C CNN
+F 2 "Transformer_SMD:Transformer_Pulse_H1100NL" H 10900 5500 50  0001 C CNN
+F 3 "https://www.mouser.ch/datasheet/2/336/pulse_07132018_PE-65728NL-1381223.pdf" H 11600 7750 50  0001 C CNN
+	1    10900 6350
+	1    0    0    -1
+$EndComp
+Text GLabel 7200 5350 2    50   Input ~ 0
+TX+
+Text GLabel 10600 6650 0    50   Input ~ 0
+TX+
+Text GLabel 10600 7050 0    50   Input ~ 0
+TX-
+Text GLabel 7200 5450 2    50   Input ~ 0
+TX-
+Text GLabel 10600 6150 0    50   Input ~ 0
+RX+
+Text GLabel 7200 5050 2    50   Input ~ 0
+RX+
+Text GLabel 10600 6550 0    50   Input ~ 0
+RX-
+Text GLabel 7200 5150 2    50   Input ~ 0
+RX-
+Text GLabel 10600 6050 0    50   Input ~ 0
+CD-
+Text GLabel 7200 4850 2    50   Input ~ 0
+CD-
+Text GLabel 10600 5650 0    50   Input ~ 0
+CD+
+Text GLabel 7200 4750 2    50   Input ~ 0
+CD+
 $EndSCHEMATC

Commit message: Work in progress
Parts:
- added C18: 47u, Capacitor_SMD:C_1210_3225Metric_Pad1.42x2.65mm_HandSolder, symbol Device:C
- added H3, H4, H5, H6, H7, H8, H9: MountingHole, ISA_BUS_16Bit:Cutline, symbol Mechanical:MountingHole
- added R22, R23, R25, R26: 510, Resistor_SMD:R_0805_2012Metric_Pad1.15x1.40mm_HandSolder, symbol Device:R
- C16, C17: value C -> 47u
Connections:
- net -9V: now also C18.2, R22.1, R23.1, R25.1, R26.1
- net GND: no longer C7.2, J1.80 (GND), U4.4 (+VOUT), U5.10 (GND), U5.16 (CDS), U5.9 (HBE)
- net at TR2.10: now also U5.7 (TX+)
- net at TR2.12: now also U5.6 (RX-), R26.2
- net at TR2.13: now also U5.3 (RX+), R25.2
- net at TR2.15: now also U5.2 (CD-), R23.2
- net at TR2.16: now also U5.1 (CD+), R22.2
- net at TR2.9: now also U5.8 (TX-)
- new net GNDA: C18.1, C7.2, U4.4 (+VOUT), U5.10 (GND), U5.16 (CDS), U5.9 (HBE)
- no-connect marks 44 -> 45
Other:
- moved on the sheet: TR2

Commit message: Work in progress
Parts:
- added R24, R27: 270, Resistor_SMD:R_0805_2012Metric_Pad1.15x1.40mm_HandSolder, symbol Device:R
- renumbered R15 to R10, R16 to R11, R17 to R12, R18 to R13, R9 to R14, R10 to R15, R11 to R16, R12 to R17, R13 to R18, R14 to R9, SW3 to SW2, SW4 to SW3, SW2 to SW4
Connections:
- net GND: now also R24.2, R27.2
- net TX+: now also R24.1
- net TX-: now also R27.1
Other:
- moved on the sheet: SW2, SW3, SW4

Commit message: Minor changes
Connections:
- net GND: now also U1.64 (AUI)
Changed lines of the file:
@@
 Connection ~ 15050 4150
 Connection ~ 15050 4650
+$Comp
+L power:GND #PWR0104
+U 1 1 6077E5A0
+P 7200 4550
+F 0 "#PWR0104" H 7200 4300 50  0001 C CNN
+F 1 "GND" H 7205 4377 50  0000 C CNN
+F 2 "" H 7200 4550 50  0001 C CNN
+F 3 "" H 7200 4550 50  0001 C CNN
+	1    7200 4550
+	0    -1   -1   0
+$EndComp
 $EndSCHEMATC

Commit message: Work in progress
Parts:
- added C19: 10n 1kV, Capacitor_SMD:C_1206_3216Metric_Pad1.42x1.75mm_HandSolder, symbol Device:C
- added Q1: PMBT2222, Package_TO_SOT_SMD:SOT-23, symbol Transistor_BJT:MMBT3904
- added R28, R29: 0, Resistor_SMD:R_0805_2012Metric_Pad1.15x1.40mm_HandSolder, symbol Device:R
- added R30: 1M, Resistor_SMD:R_0805_2012Metric_Pad1.15x1.40mm_HandSolder, symbol Device:R
- added R31: 1K, Resistor_SMD:R_0805_2012Metric_Pad1.15x1.40mm_HandSolder, symbol Device:R
- C3, C4: value 1nF 2kV -> 100n; footprint Capacitor_SMD:C_1206_3216Metric_Pad1.42x1.75mm_HandSolder -> Capacitor_SMD:C_0805_2012Metric_Pad1.15x1.40mm_HandSolder
- C5, C6: value 1nF 2kV -> 39p 2kV
Connections:
- net GND: now also Q1.2 (E), R28.2, R29.2; no longer C5.1, C6.2, H1.1, H2.1, J2.SH, J3.2 (Ext), U4.1 (-VIN)
- net GNDA: now also J3.2 (Ext), C19.1, R30.1
- net at U1.60 (LEDBNC): now also R31.2
- net at J2.1, TR1.16 (TX+): now also C6.1
- net at J2.2, TR1.14 (TX-): now also C5.1
- net at TR1.10 (C_RX): no longer C5.2
- net at TR1.15 (C_TX): no longer C6.1
- new net: Q1.3 (C), U4.1 (-VIN)
- new net: Q1.1 (B), R31.1
- new net Earth: C19.2, C5.2, C6.2, H1.1, H2.1, J2.SH, R28.1, R29.1, R30.2
- no-connect marks 45 -> 47
Other:
- moved on the sheet: C18, U4

Commit message: Work in progress
Parts:
- removed J3: BNC, Connector_Coaxial:BNC_Amphenol_B6252HB-NPP3G-50_Horizontal, symbol Connector:Conn_Coaxial
- added H10: MountingHole, ISA_BUS_16Bit:Cutline, symbol Mechanical:MountingHole
- added J3: BNC, Coax:BNC_shield, symbol 10Base2:BNC_shield
- renumbered R25 to R24, R26 to R25, R24 to R26
Connections:
- net Earth: now also J3.3
- net GNDA: now also J3.2
- net at D1.2 (A), U5.14 (RXI): now also J3.1
Other:
- moved on the sheet: H3, H4, H5, H6, H7, H8, H9
Changed lines of the file:
@@
 EESchema Schematic File Version 4
-LIBS:NE2000-cache
 EELAYER 30 0
 EELAYER END
@@
 Wire Wire Line
 	14350 6200 14350 6100
-$Comp
-L Connector:Conn_Coaxial J3
-U 1 1 6081E2FE
-P 14850 6100
-F 0 "J3" H 14950 6075 50  0000 L CNN
-F 1 "BNC" H 14950 5984 50  0000 L CNN
-F 2 "Connector_Coaxial:BNC_Amphenol_B6252HB-NPP3G-50_Horizontal" H 14850 6100 50  0001 C CNN
-F 3 "https://www.mouser.ch/datasheet/2/18/031_71052_customer_drawing-1820911.pdf" H 14850 6100 50  0001 C CNN
-	1    14850 6100
-	1    0    0    -1
-$EndComp
 Wire Wire Line
 	14350 6100 14650 6100
@@
 L Mechanical:MountingHole H9
 U 1 1 607109EC
-P 600 11100
-F 0 "H9" H 700 11146 50  0000 L CNN
-F 1 "MountingHole" H 700 11055 50  0000 L CNN
-F 2 "ISA_BUS_16Bit:Cutline" H 600 11100 50  0001 C CNN
-F 3 "~" H 600 11100 50  0001 C CNN
-	1    600  11100
-	1    0    0    -1
-$EndComp
-$Comp
-L Mechanical:MountingHole H8
-U 1 1 6071198A
 P 600 10900
-F 0 "H8" H 700 10946 50  0000 L CNN
+F 0 "H9" H 700 10946 50  0000 L CNN
 F 1 "MountingHole" H 700 10855 50  0000 L CNN
 F 2 "ISA_BUS_16Bit:Cutline" H 600 10900 50  0001 C CNN
@@
 $EndComp
 $Comp
-L Mechanical:MountingHole H7
-U 1 1 60712463
+L Mechanical:MountingHole H8
+U 1 1 6071198A
 P 600 10700
-F 0 "H7" H 700 10746 50  0000 L CNN
+F 0 "H8" H 700 10746 50  0000 L CNN
 F 1 "MountingHole" H 700 10655 50  0000 L CNN
 F 2 "ISA_BUS_16Bit:Cutline" H 600 10700 50  0001 C CNN
@@
 $EndComp
 $Comp
-L Mechanical:MountingHole H6
-U 1 1 60713BDB
+L Mechanical:MountingHole H7
+U 1 1 60712463
 P 600 10500
-F 0 "H6" H 700 10546 50  0000 L CNN
+F 0 "H7" H 700 10546 50  0000 L CNN
 F 1 "MountingHole" H 700 10455 50  0000 L CNN
 F 2 "ISA_BUS_16Bit:Cutline" H 600 10500 50  0001 C CNN
@@
 $EndComp
 $Comp
+L Mechanical:MountingHole H6
+U 1 1 60713BDB
+P 600 10300
+F 0 "H6" H 700 10346 50  0000 L CNN
+F 1 "MountingHole" H 700 10255 50  0000 L CNN
+F 2 "ISA_BUS_16Bit:Cutline" H 600 10300 50  0001 C CNN
+F 3 "~" H 600 10300 50  0001 C CNN
+	1    600  10300
+	1    0    0    -1
+$EndComp
+$Comp
 L Mechanical:MountingHole H3
 U 1 1 607157E2
+P 600 9700
+F 0 "H3" H 700 9746 50  0000 L CNN
+F 1 "MountingHole" H 700 9655 50  0000 L CNN
+F 2 "ISA_BUS_16Bit:Cutline" H 600 9700 50  0001 C CNN
+F 3 "~" H 600 9700 50  0001 C CNN
+	1    600  9700
+	1    0    0    -1
+$EndComp
+$Comp
+L Mechanical:MountingHole H4
+U 1 1 60724CD1
 P 600 9900
-F 0 "H3" H 700 9946 50  0000 L CNN
+F 0 "H4" H 700 9946 50  0000 L CNN
 F 1 "MountingHole" H 700 9855 50  0000 L CNN
 F 2 "ISA_BUS_16Bit:Cutline" H 600 9900 50  0001 C CNN
@@
 $EndComp
 $Comp
-L Mechanical:MountingHole H4
-U 1 1 60724CD1
+L Mechanical:MountingHole H5
+U 1 1 60737F12
 P 600 10100
-F 0 "H4" H 700 10146 50  0000 L CNN
+F 0 "H5" H 700 10146 50  0000 L CNN
 F 1 "MountingHole" H 700 10055 50  0000 L CNN
 F 2 "ISA_BUS_16Bit:Cutline" H 600 10100 50  0001 C CNN
 F 3 "~" H 600 10100 50  0001 C CNN
 	1    600  10100
-	1    0    0    -1
-$EndComp
-$Comp
-L Mechanical:MountingHole H5
-U 1 1 60737F12
-P 600 10300
-F 0 "H5" H 700 10346 50  0000 L CNN
-F 1 "MountingHole" H 700 10255 50  0000 L CNN
-F 2 "ISA_BUS_16Bit:Cutline" H 600 10300 50  0001 C CNN
-F 3 "~" H 600 10300 50  0001 C CNN
-	1    600  10300
 	1    0    0    -1
 $EndComp
@@
 $EndComp
 $Comp
-L Device:R R25
+L Device:R R24
 U 1 1 6077B404
 P 12100 5800
-F 0 "R25" H 12170 5846 50  0000 L CNN
+F 0 "R24" H 12170 5846 50  0000 L CNN
 F 1 "510" H 12170 5755 50  0000 L CNN
 F 2 "Resistor_SMD:R_0805_2012Metric_Pad1.15x1.40mm_HandSolder" V 12030 5800 50  0001 C CNN
@@
 $EndComp
 $Comp
-L Device:R R26
+L Device:R R25
 U 1 1 6077B61B
 P 12400 5800
-F 0 "R26" H 12470 5846 50  0000 L CNN
+F 0 "R25" H 12470 5846 50  0000 L CNN
 F 1 "510" H 12470 5755 50  0000 L CNN
 F 2 "Resistor_SMD:R_0805_2012Metric_Pad1.15x1.40mm_HandSolder" V 12330 5800 50  0001 C CNN
@@
 $EndComp
 $Comp
-L Device:R R24
+L Device:R R26
 U 1 1 6072BB38
 P 10300 7400
-F 0 "R24" H 10370 7446 50  0000 L CNN
+F 0 "R26" H 10370 7446 50  0000 L CNN
 F 1 "270" H 10370 7355 50  0000 L CNN
 F 2 "Resistor_SMD:R_0805_2012Metric_Pad1.15x1.40mm_HandSolder" V 10230 7400 50  0001 C CNN
@@
 Wire Wire Line
 	8400 8850 8500 8850
+$Comp
+L 10Base2:BNC_shield J3
+U 1 1 607A8534
+P 14850 6100
+F 0 "J3" H 14850 6356 50  0000 C CNN
+F 1 "BNC" H 14850 6265 50  0000 C CNN
+F 2 "Coax:BNC_shield" H 15350 6550 50  0001 C CNN
+F 3 "https://www.mouser.ch/datasheet/2/18/031_71052_customer_drawing-1820911.pdf" H 15350 6550 50  0001 C CNN
+	1    14850 6100
+	1    0    0    -1
+$EndComp
+$Comp
+L power:Earth #PWR0119
+U 1 1 607B29CE
+P 15050 6100
+F 0 "#PWR0119" H 15050 5850 50  0001 C CNN
+F 1 "Earth" H 15050 5950 50  0001 C CNN
+F 2 "" H 15050 6100 50  0001 C CNN
+F 3 "~" H 15050 6100 50  0001 C CNN
+	1    15050 6100
+	0    -1   -1   0
+$EndComp
+$Comp
+L Mechanical:MountingHole H10
+U 1 1 60839C70
+P 600 11100
+F 0 "H10" H 700 11146 50  0000 L CNN
+F 1 "MountingHole" H 700 11055 50  0000 L CNN
+F 2 "ISA_BUS_16Bit:Cutline" H 600 11100 50  0001 C CNN
+F 3 "~" H 600 11100 50  0001 C CNN
+	1    600  11100
+	1    0    0    -1
+$EndComp
 $EndSCHEMATC

Commit message: Work in progress
Parts:
- removed U4: IL1209S, Converter_DCDC:Converter_DCDC_muRata_CRE1xxxxxx3C_THT, symbol Regulator_Switching:CRE1S0305S3C
- added U4: IL1209S, IL1209S, symbol Samac:IL1209S
- C1, C2: Mouser (none) -> 80-C0805C220K3HACTU
- C10, C11, C12, C13, C14, C15, C3, C4, C7, C8, C9: Mouser (none) -> 80-C0805C104M5R
- C16, C17, C18: Mouser (none) -> 81-GRM32EC81C476KE5L
- C19: Mouser (none) -> 710-885342208021
- C5, C6: Mouser (none) -> 81-GRM31A7U3D390JW1D
- D1: value 1N4150 -> BAS16; Mouser (none) -> 841-BAS16GWJ
- J2: Mouser (none) -> 523-RJHSE-5481
- J3: Mouser (none) -> 538-73137-5003
- Q1: Mouser (none) -> 771-PMBT2222A-T/R
- R1: Mouser (none) -> 652-CR0805FX-2702ELF
- R10, R11, R12, R13, R14, R15, R16, R17, R18, R19, R20, R5, R6, R7, R8, R9: Mouser (none) -> 652-CR0805-JW-103ELF
- R2, R3: Mouser (none) -> 652-CR0805FX-4700ELF
- R21, R31: Mouser (none) -> 652-CR0805FX-1001ELF
- R22, R23, R24, R25: Mouser (none) -> 603-RC0805JR-07510RL
- R26, R27: Mouser (none) -> 71-CRCW0805270RJNEA
- R28, R29: Mouser (none) -> 603-RC0805JR-070RL
- R30: Mouser (none) -> 652-CMP0805AFX-1004L
- R4: Mouser (none) -> 652-CR0805FX-2000ELF
- SW1: Mouser (none) -> 774-2104MS
- SW2: Mouser (none) -> 774-2103MS
- SW3, SW5: Mouser (none) -> 774-2102MS
- SW4: Mouser (none) -> 774-2105MS
- TR1: Mouser (none) -> 652-PT61017PEL
- TR2: Mouser (none) -> 673-PE-65728NL
- U2: Mouser (none) -> 556-A93C46DNSH-B
- U3: Mouser (none) -> 649-DILB32P223TLF
- Y1: Mouser (none) -> 815-ABL-20-B2
Connections:
- net +12V: now also U4.2 (+VIN)
- net -9V: now also U4.3 (-VOUT)
- net GNDA: now also U4.4 (+VOUT)
- net at Q1.3 (C): now also U4.1 (-VIN)
Other:
- moved on the sheet: C18

Commit message: Use different DC/DC converter
Parts:
- U4: footprint IL1209S -> Samac:DC_DC_12to9
Changed lines of the file:
@@
 F 0 "U4" H 10728 8546 50  0000 L CNN
 F 1 "IL1209S" H 10728 8455 50  0000 L CNN
-F 2 "IL1209S" H 10750 8750 50  0001 L CNN
+F 2 "Samac:DC_DC_12to9" H 10750 8750 50  0001 L CNN
 F 3 "https://componentsearchengine.com/Datasheets/2/IL1209S.pdf" H 10750 8650 50  0001 L CNN
 F 4 "Isolated DC/DC Converters DC-DC, 2W, unreg., single output, SIP" H 10750 8550 50  0001 L CNN "Description"
